File: aiot_pcb_play.kicad_pcb (KiCad board)
At the start: 4 copper layers, 56 x 85 mm, 11 parts, among them J1 10_pin_swd_connector, J2 Tag-Connect, U2 16_pin_header

Commit message: #1 Made changes to the PCB
Parts:
- BT1: renamed from REF**; value BatteryHolder_MPD_BC2AAPC_2xAA -> Battery_Cell
- renumbered nRF52833 to U1, Dusty to U3
Connections:
- U1 pad 8: Net-(U1-Pad8) -> P0.31
- U2 pad 15: Net-(U1-Pad8) -> P0.31
- U3 pad 33: unconnected-(U3-Pad33) -> VDD
- U3 pad 37: unconnected-(U3-Pad37) -> GND
- U3 pad 39: unconnected-(U3-Pad39) -> P0.31
Routing:
- net P0.31: track 0.00 -> 50.0 mm, vias 0 -> 2
- net Net-(U1-Pad8): track 32.2 -> 0.00 mm, vias 1 -> 0
- net VDD: track 146.6 -> 131.5 mm
- net GND: track 15.1 -> 16.9 mm, vias 15 -> 16
- net Net-(J1-Pad4): track 42.3 -> 43.1 mm
Other:
- board text added: "(TIMEn)"
- board text added: "Dusty"
- board text added: "Play v1.1"
- board text added: "nRF52833"
- board text removed: "Play v1.0"

Commit message: #1 Fix: Mounting holes not detected by PCB manufacturer
Eurocircuits was not registering the Mounting holes on the PCB, so I changed the footprint
Parts:
- added REF**: MountingHole_2.7mm, MountingHole:MountingHole_2.7mm, F.Cu at (177.5, 131.5)
- added REF**: MountingHole_2.7mm, MountingHole:MountingHole_2.7mm, F.Cu at (177.5, 73.5)
- added REF**: MountingHole_2.7mm, MountingHole:MountingHole_2.7mm, F.Cu at (128.5, 131.5)
- added REF**: MountingHole_2.7mm, MountingHole:MountingHole_2.7mm, F.Cu at (128.5, 73.5)
Other:
- outline, holes or cut-outs redrawn
Changed lines of the file:
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@@
       (net 1 "GND") (pinfunction "GND") (pintype "input"))
+  )
+  (footprint "MountingHole:MountingHole_2.7mm" (layer "F.Cu")
+    (at 177.5 131.5)
+    (descr "Mounting Hole 2.7mm, no annular")
+    (tags "mounting hole 2.7mm no annular")
+    (attr exclude_from_pos_files exclude_from_bom)
+    (fp_text reference "REF**" (at 6 0.15) (layer "F.SilkS") hide
+      (effects (font (size 1 1) (thickness 0.15)))
+    )
+    (fp_text value "MountingHole_2.7mm" (at 0 3.7) (layer "F.Fab")
+      (effects (font (size 1 1) (thickness 0.15)))
+    )
+    (fp_text user "${REFERENCE}" (at 0.3 0) (layer "F.Fab")
+      (effects (font (size 1 1) (thickness 0.15)))
+    )
+    (fp_circle (center 0 0) (end 2.7 0) (layer "Cmts.User") (width 0.15) (fill none))
+    (fp_circle (center 0 0) (end 2.95 0) (layer "F.CrtYd") (width 0.05) (fill none))
+    (pad "" np_thru_hole circle locked (at 0 0) (size 2.7 2.7) (drill 2.7) (layers *.Cu *.Mask))
   )
   (footprint "Capacitor_SMD:C_0603_1608Metric" (layer "F.Cu")
@@
       (rotate (xyz 0 0 0))
     )
+  )
+  (footprint "MountingHole:MountingHole_2.7mm" (layer "F.Cu")
+    (at 177.5 73.5)
+    (descr "Mounting Hole 2.7mm, no annular")
+    (tags "mounting hole 2.7mm no annular")
+    (attr exclude_from_pos_files exclude_from_bom)
+    (fp_text reference "REF**" (at 5.95 0.15) (layer "F.SilkS") hide
+      (effects (font (size 1 1) (thickness 0.15)))
+    )
+    (fp_text value "MountingHole_2.7mm" (at 0 3.7) (layer "F.Fab")
+      (effects (font (size 1 1) (thickness 0.15)))
+    )
+    (fp_text user "${REFERENCE}" (at 0.3 0) (layer "F.Fab")
+      (effects (font (size 1 1) (thickness 0.15)))
+    )
+    (fp_circle (center 0 0) (end 2.7 0) (layer "Cmts.User") (width 0.15) (fill none))
+    (fp_circle (center 0 0) (end 2.95 0) (layer "F.CrtYd") (width 0.05) (fill none))
+    (pad "" np_thru_hole circle locked (at 0 0) (size 2.7 2.7) (drill 2.7) (layers *.Cu *.Mask))
+  )
+  (footprint "MountingHole:MountingHole_2.7mm" (layer "F.Cu")
+    (at 128.5 131.5)
+    (descr "Mounting Hole 2.7mm, no annular")
+    (tags "mounting hole 2.7mm no annular")
+    (attr exclude_from_pos_files exclude_from_bom)
+    (fp_text reference "REF**" (at -6.25 -0.05) (layer "F.SilkS") hide
+      (effects (font (size 1 1) (thickness 0.15)))
+    )
+    (fp_text value "MountingHole_2.7mm" (at 0 3.7) (layer "F.Fab")
+      (effects (font (size 1 1) (thickness 0.15)))
+    )
+    (fp_text user "${REFERENCE}" (at 0.3 0) (layer "F.Fab")
+      (effects (font (size 1 1) (thickness 0.15)))
+    )
+    (fp_circle (center 0 0) (end 2.7 0) (layer "Cmts.User") (width 0.15) (fill none))
+    (fp_circle (center 0 0) (end 2.95 0) (layer "F.CrtYd") (width 0.05) (fill none))
+    (pad "" np_thru_hole circle locked (at 0 0) (size 2.7 2.7) (drill 2.7) (layers *.Cu *.Mask))
   )
   (footprint "iot_lib:tag-connect_10_pins_no_hooks" (layer "F.Cu")
@@
     (pad "1" smd circle (at 0.025 0.025) (size 2 2) (layers "F.Cu" "F.Paste" "F.Mask")
       (net 34 "Net-(TP2-Pad1)") (pinfunction "1") (pintype "passive"))
+  )
+  (footprint "MountingHole:MountingHole_2.7mm" (layer "F.Cu")
+    (at 128.5 73.5)
+    (descr "Mounting Hole 2.7mm, no annular")
+    (tags "mounting hole 2.7mm no annular")
+    (attr exclude_from_pos_files exclude_from_bom)
+    (fp_text reference "REF**" (at -6.95 0.3) (layer "F.SilkS") hide
+      (effects (font (size 1 1) (thickness 0.15)))
+    )
+    (fp_text value "MountingHole_2.7mm" (at 0 3.7) (layer "F.Fab")
+      (effects (font (size 1 1) (thickness 0.15)))
+    )
+    (fp_text user "${REFERENCE}" (at 0.3 0) (layer "F.Fab")
+      (effects (font (size 1 1) (thickness 0.15)))
+    )
+    (fp_circle (center 0 0) (end 2.7 0) (layer "Cmts.User") (width 0.15) (fill none))
+    (fp_circle (center 0 0) (end 2.95 0) (layer "F.CrtYd") (width 0.05) (fill none))
+    (pad "" np_thru_hole circle locked (at 0 0) (size 2.7 2.7) (drill 2.7) (layers *.Cu *.Mask))
   )
   (footprint "Battery:BatteryHolder_MPD_BC2AAPC_2xAA" (layer "B.Cu")
@@
   (gr_line (start 151.57 106.84) (end 151.57 93.9) (layer "F.SilkS") (width 0.3))
   (gr_circle (center 177.5 131.5) (end 180.5 131.5) (layer "F.SilkS") (width 0.1) (fill none))
-  (gr_circle (center 177.5 131.5) (end 178.85 131.5) (layer "Edge.Cuts") (width 0.1) (fill none))
   (gr_line (start 128 50) (end 134.5 50) (layer "Edge.Cuts") (width 0.15))
-  (gr_circle (center 128.5 131.5) (end 129.85 131.5) (layer "Edge.Cuts") (width 0.1) (fill none))
   (gr_line (start 150.6 50) (end 150.6 56.3) (layer "Edge.Cuts") (width 0.15))
   (gr_arc (start 128 135) (mid 125.87868 134.12132) (end 125 132) (layer "Edge.Cuts") (width 0.15))
-  (gr_circle (center 128.5 73.5) (end 129.85 73.5) (layer "Edge.Cuts") (width 0.1) (fill none))
   (gr_line (start 161.7 50) (end 161.7 54.4) (layer "Edge.Cuts") (width 0.15))
   (gr_arc (start 181 132) (mid 180.12132 134.12132) (end 178 135) (layer "Edge.Cuts") (width 0.15))
@@
   (gr_line (start 181 53) (end 181 132) (layer "Edge.Cuts") (width 0.15))
   (gr_line (start 134.5 56.3) (end 134.5 50) (layer "Edge.Cuts") (width 0.15))
-  (gr_circle (center 177.5 73.5) (end 178.85 73.5) (layer "Edge.Cuts") (width 0.1) (fill none))
   (gr_line (start 125 53) (end 125 132) (layer "Edge.Cuts") (width 0.15))
   (gr_line (start 150.6 50) (end 161.7 50) (layer "Edge.Cuts") (width 0.15))
